File: projects/pihat-template-master-3edcb619cb61f66af69215d6eb82650f2881d374/hardware/jvm_options.sch (KiCad schematic (older format))
At the start: 7 parts

Commit message: Started placement of MAXM17503
Parts:
- removed U?: MAXM17503, symbol MAXM17503-RESCUE-pihat_template
- removed U?: MAXM17503, symbol MAXM17503
- added C10: 11nF, Capacitors_SMD:C_0603_HandSoldering, symbol C
- added C11: 2.2uF, Capacitors_SMD:C_1206_HandSoldering, symbol C
- added C12: DNI, Capacitors_SMD:C_0603_HandSoldering, symbol C
- added C13: 22uF, Capacitors_SMD:C_1210_HandSoldering, symbol C
- added C9: 2.2uf, Capacitors_SMD:C_1206_HandSoldering, symbol C
- added R18: 191k, Resistors_SMD:R_0603_HandSoldering, symbol R
- added R19: 42.2k, Resistors_SMD:R_0603_HandSoldering, symbol R
- added R20, R21: 10k, Resistors_SMD:R_0603_HandSoldering, symbol R
- added R22: .1, Resistors_SMD:R_0603_HandSoldering, symbol R
- added U6: MAXM17503, jvm:MAXM17503, symbol MAXM17503
- R13: renamed from R?; value R -> 3.3M; footprint (none) -> Resistors_SMD:R_0603_HandSoldering
- R14, R15, R16: renamed from R?; value R -> 100K; footprint (none) -> Resistors_SMD:R_0603_HandSoldering
- R17: renamed from R?; value R -> 26.7k; footprint (none) -> Resistors_SMD:R_0603_HandSoldering
Connections:
- net labels added: +3.3V, +5V_Output, RawPower, SCL, SDA
- net labels removed: +24V
- wire segments 0 -> 67
- no-connect marks 0 -> 2
