File: projects/pihat-template-master-3edcb619cb61f66af69215d6eb82650f2881d374/hardware/pihat_template.sch (KiCad schematic (older format))
At the start: 30 parts, among them P1 CONN_01X02, P2 CONN_01X02, P3 Raspberry_Pi_+_Conn, U1 LM3489, U2 CAT24C32HU4I-GT3, U3 FDC5614P, U4 LM1117IMPX-ADJ

Commit message: Started placement of MAXM17503
Parts:
- removed U?: MAXM17503, symbol MAXM17503-RESCUE-pihat_template
Connections:
- net SDA: now reaches P3.3 (GPIO2/I2C1_SDA)
- net SCL: now reaches P3.5 (GPIO3/I2C1_SCL)
- no-connect marks 0 -> 27
