File: projects/myhat/hardware/pihat_template.sch (KiCad schematic (older format))
At the start: 29 parts, among them P1 CONN_01X02, P2 CONN_01X02, P3 Raspberry_Pi_+_Conn, U1 LM3489, U2 CAT24C32HU4I-GT3, U3 FDC5614P, U4 LM1117IMPX-ADJ

Commit message: updated hat_options
Changed lines of the file:
@@
 F5 "Bat_-" I L 7450 7050 60
 F6 "Ext_-" I L 7450 7300 60
-F7 "24_V" O R 9500 7150 60
-F8 "5_V" O R 9500 7450 60
+F7 "5_V" O R 9500 7450 60
 $EndSheet
 $EndSCHEMATC
